File: I2C-7311.brd (EAGLE design)
At the start: 106 x 100 mm, 79 parts, among them IC1 MAX7311, Q0 P-FET, Q1 P-FET, Q10 P-FET, Q11 P-FET, Q12 P-FET, Q13 P-FET, Q14 P-FET, Q15 P-FET, Q2 P-FET, Q3 P-FET, Q4 P-FET, Q5 P-FET, Q6 P-FET, Q7 P-FET, Q8 P-FET, Q9 P-FET, SW1 A0, SW2 A1, SW3 A2

Commit message: V3.1 again
Parts:
- turned Q0 to 90 degrees
- turned Q1 to 90 degrees
- turned Q10 to 90 degrees
- turned Q11 to 90 degrees
- turned Q12 to 90 degrees
- turned Q13 to 90 degrees
- turned Q14 to 90 degrees
- turned Q15 to 90 degrees
- turned Q2 to 90 degrees
- turned Q3 to 90 degrees
- turned Q4 to 90 degrees
- turned Q5 to 90 degrees
- turned Q6 to 90 degrees
- turned Q7 to 90 degrees
- turned Q8 to 90 degrees
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Changed lines of the file:
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@@
 <grid distance="50" unitdist="mil" unit="mil" style="dots" multiple="2" display="yes" altdistance="25" altunitdist="mil" altunit="mil"/>
 <layers>
-<layer number="1" name="Top" color="4" fill="1" visible="yes" active="yes"/>
-<layer number="16" name="Bottom" color="2" fill="1" visible="yes" active="yes"/>
+<layer number="1" name="Top" color="4" fill="1" visible="no" active="yes"/>
+<layer number="16" name="Bottom" color="2" fill="1" visible="no" active="yes"/>
 <layer number="17" name="Pads" color="23" fill="1" visible="yes" active="yes"/>
 <layer number="18" name="Vias" color="29" fill="1" visible="yes" active="yes"/>
@@
 <element name="LED3" library="SPCoast" package="0603-LED" value="Y" x="81.28" y="34.29" smashed="yes" rot="R90"/>
 <element name="LED4" library="SPCoast" package="0603-LED" value="Y" x="77.47" y="34.29" smashed="yes" rot="R90"/>
-<element name="Q0" library="SPCoast" package="SOT23" value="P-FET" x="88.9" y="38.735" smashed="yes" rot="R180">
-<attribute name="NAME" x="90.424" y="38.481" size="0.254" layer="25" ratio="11" rot="R270"/>
-</element>
-<element name="Q1" library="SPCoast" package="SOT23" value="P-FET" x="85.09" y="38.735" smashed="yes" rot="R180">
-<attribute name="NAME" x="86.614" y="38.481" size="0.254" layer="25" ratio="11" rot="R270"/>
-</element>
-<element name="Q2" library="SPCoast" package="SOT23" value="P-FET" x="81.28" y="38.735" smashed="yes" rot="R180">
-<attribute name="NAME" x="82.804" y="38.481" size="0.254" layer="25" ratio="11" rot="R270"/>
-</element>
-<element name="Q3" library="SPCoast" package="SOT23" value="P-FET" x="77.47" y="38.735" smashed="yes" rot="R180">
-<attribute name="NAME" x="78.994" y="38.481" size="0.254" layer="25" ratio="11" rot="R270"/>
+<element name="Q0" library="SPCoast" package="SOT23" value="P-FET" x="88.9" y="38.735" smashed="yes" rot="R90">
+<attribute name="NAME" x="88.646" y="37.211" size="0.254" layer="25" ratio="11" rot="R180"/>
+</element>
+<element name="Q1" library="SPCoast" package="SOT23" value="P-FET" x="85.09" y="38.735" smashed="yes" rot="R90">
+<attribute name="NAME" x="84.836" y="37.211" size="0.254" layer="25" ratio="11" rot="R180"/>
+</element>
+<element name="Q2" library="SPCoast" package="SOT23" value="P-FET" x="81.28" y="38.735" smashed="yes" rot="R90">
+<attribute name="NAME" x="81.026" y="37.211" size="0.254" layer="25" ratio="11" rot="R180"/>
+</element>
+<element name="Q3" library="SPCoast" package="SOT23" value="P-FET" x="77.47" y="38.735" smashed="yes" rot="R90">
+<attribute name="NAME" x="77.216" y="37.211" size="0.254" layer="25" ratio="11" rot="R180"/>
 </element>
 <element name="R7" library="SPCoast" package="0805-RES" value="2K0" x="86.995" y="36.195" smashed="yes" rot="R90">
@@
 <element name="LED6" library="SPCoast" package="0603-LED" value="Y" x="59.69" y="34.29" smashed="yes" rot="R90"/>
 <element name="LED7" library="SPCoast" package="0603-LED" value="Y" x="55.88" y="34.29" smashed="yes" rot="R90"/>
-<element name="Q4" library="SPCoast" package="SOT23" value="P-FET" x="67.31" y="38.735" smashed="yes" rot="R180">
-<attribute name="NAME" x="68.834" y="38.481" size="0.254" layer="25" ratio="11" rot="R270"/>
-</element>
-<element name="Q5" library="SPCoast" package="SOT23" value="P-FET" x="63.5" y="38.735" smashed="yes" rot="R180">
-<attribute name="NAME" x="65.024" y="38.481" size="0.254" layer="25" ratio="11" rot="R270"/>
-</element>
-<element name="Q6" library="SPCoast" package="SOT23" value="P-FET" x="59.69" y="38.735" smashed="yes" rot="R180">
-<attribute name="NAME" x="61.214" y="38.481" size="0.254" layer="25" ratio="11" rot="R270"/>
-</element>
-<element name="Q7" library="SPCoast" package="SOT23" value="P-FET" x="55.88" y="38.735" smashed="yes" rot="R180">
-<attribute name="NAME" x="57.404" y="38.481" size="0.254" layer="25" ratio="11" rot="R270"/>
+<element name="Q4" library="SPCoast" package="SOT23" value="P-FET" x="67.31" y="38.735" smashed="yes" rot="R90">
+<attribute name="NAME" x="67.056" y="37.211" size="0.254" layer="25" ratio="11" rot="R180"/>
+</element>
+<element name="Q5" library="SPCoast" package="SOT23" value="P-FET" x="63.5" y="38.735" smashed="yes" rot="R90">
+<attribute name="NAME" x="63.246" y="37.211" size="0.254" layer="25" ratio="11" rot="R180"/>
+</element>
+<element name="Q6" library="SPCoast" package="SOT23" value="P-FET" x="59.69" y="38.735" smashed="yes" rot="R90">
+<attribute name="NAME" x="59.436" y="37.211" size="0.254" layer="25" ratio="11" rot="R180"/>
+</element>
+<element name="Q7" library="SPCoast" package="SOT23" value="P-FET" x="55.88" y="38.735" smashed="yes" rot="R90">
+<attribute name="NAME" x="55.626" y="37.211" size="0.254" layer="25" ratio="11" rot="R180"/>
 </element>
 <element name="R11" library="SPCoast" package="0805-RES" value="2K0" x="65.405" y="36.195" smashed="yes" rot="R90">
@@
 </element>
 <element name="LED11" library="SPCoast" package="0603-LED" value="Y" x="34.29" y="34.29" smashed="yes" rot="R90"/>
-<element name="Q8" library="SPCoast" package="SOT23" value="P-FET" x="45.72" y="38.735" smashed="yes" rot="R180">
-<attribute name="NAME" x="47.244" y="38.481" size="0.254" layer="25" ratio="11" rot="R270"/>
-</element>
-<element name="Q9" library="SPCoast" package="SOT23" value="P-FET" x="41.91" y="38.735" smashed="yes" rot="R180">
-<attribute name="NAME" x="43.434" y="38.481" size="0.254" layer="25" ratio="11" rot="R270"/>
-</element>
-<element name="Q10" library="SPCoast" package="SOT23" value="P-FET" x="38.1" y="38.735" smashed="yes" rot="R180">
-<attribute name="NAME" x="39.624" y="38.481" size="0.254" layer="25" ratio="11" rot="R270"/>
-</element>
-<element name="Q11" library="SPCoast" package="SOT23" value="P-FET" x="34.29" y="38.735" smashed="yes" rot="R180">
-<attribute name="NAME" x="35.814" y="38.481" size="0.254" layer="25" ratio="11" rot="R270"/>
+<element name="Q8" library="SPCoast" package="SOT23" value="P-FET" x="45.72" y="38.735" smashed="yes" rot="R90">
+<attribute name="NAME" x="45.466" y="37.211" size="0.254" layer="25" ratio="11" rot="R180"/>
+</element>
+<element name="Q9" library="SPCoast" package="SOT23" value="P-FET" x="41.91" y="38.735" smashed="yes" rot="R90">
+<attribute name="NAME" x="41.656" y="37.211" size="0.254" layer="25" ratio="11" rot="R180"/>
+</element>
+<element name="Q10" library="SPCoast" package="SOT23" value="P-FET" x="38.1" y="38.735" smashed="yes" rot="R90">
+<attribute name="NAME" x="37.846" y="37.211" size="0.254" layer="25" ratio="11" rot="R180"/>
+</element>
+<element name="Q11" library="SPCoast" package="SOT23" value="P-FET" x="34.29" y="38.735" smashed="yes" rot="R90">
+<attribute name="NAME" x="34.036" y="37.211" size="0.254" layer="25" ratio="11" rot="R180"/>
 </element>
 <element name="R15" library="SPCoast" package="0805-RES" value="2K0" x="43.815" y="36.195" smashed="yes" rot="R90">
@@
 <element name="LED14" library="SPCoast" package="0603-LED" value="Y" x="16.51" y="34.29" smashed="yes" rot="R90"/>
 <element name="LED15" library="SPCoast" package="0603-LED" value="Y" x="12.7" y="34.29" smashed="yes" rot="R90"/>
-<element name="Q12" library="SPCoast" package="SOT23" value="P-FET" x="24.13" y="38.735" smashed="yes" rot="R180">
-<attribute name="NAME" x="25.654" y="38.481" size="0.254" layer="25" ratio="11" rot="R270"/>
-</element>
-<element name="Q13" library="SPCoast" package="SOT23" value="P-FET" x="20.32" y="38.735" smashed="yes" rot="R180">
-<attribute name="NAME" x="21.844" y="38.481" size="0.254" layer="25" ratio="11" rot="R270"/>
-</element>
-<element name="Q14" library="SPCoast" package="SOT23" value="P-FET" x="16.51" y="38.735" smashed="yes" rot="R180">
-<attribute name="NAME" x="18.034" y="38.481" size="0.254" layer="25" ratio="11" rot="R270"/>
-</element>
-<element name="Q15" library="SPCoast" package="SOT23" value="P-FET" x="12.7" y="38.735" smashed="yes" rot="R180">
-<attribute name="NAME" x="14.224" y="38.481" size="0.254" layer="25" ratio="11" rot="R270"/>
+<element name="Q12" library="SPCoast" package="SOT23" value="P-FET" x="24.13" y="38.735" smashed="yes" rot="R90">
+<attribute name="NAME" x="23.876" y="37.211" size="0.254" layer="25" ratio="11" rot="R180"/>
+</element>
+<element name="Q13" library="SPCoast" package="SOT23" value="P-FET" x="20.32" y="38.735" smashed="yes" rot="R90">
+<attribute name="NAME" x="20.066" y="37.211" size="0.254" layer="25" ratio="11" rot="R180"/>
+</element>
+<element name="Q14" library="SPCoast" package="SOT23" value="P-FET" x="16.51" y="38.735" smashed="yes" rot="R90">
+<attribute name="NAME" x="16.256" y="37.211" size="0.254" layer="25" ratio="11" rot="R180"/>
+</element>
+<element name="Q15" library="SPCoast" package="SOT23" value="P-FET" x="12.7" y="38.735" smashed="yes" rot="R90">
+<attribute name="NAME" x="12.446" y="37.211" size="0.254" layer="25" ratio="11" rot="R180"/>
 </element>
 <element name="R22" library="SPCoast" package="0805-RES" value="2K0" x="22.225" y="36.195" smashed="yes" rot="R90">

Commit message: SPCoast lbr footprint update
Parts:
- IOB1, IOB2, IOB3: value CONNECTOR-IO4-IOBCLEAN -> CONNECTOR-IO4-IOBNOBSILK; device SPCoast:IOB-IO4-CLEAN -> SPCoast:IOB-IO4-NOBOTSILK
- IOB4: value CONNECTOR-IO4-IOBBARE -> CONNECTOR-IO4-IOBFULL
- moved U$1 10.2 mm to (81.9, 82.7)
- renumbered FID1 to FID-UL, FID2 to FID-LR
Changed lines of the file:
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@@
 <grid distance="50" unitdist="mil" unit="mil" style="dots" multiple="2" display="yes" altdistance="25" altunitdist="mil" altunit="mil"/>
 <layers>
-<layer number="1" name="Top" color="4" fill="1" visible="no" active="yes"/>
-<layer number="16" name="Bottom" color="2" fill="1" visible="no" active="yes"/>
+<layer number="1" name="Top" color="4" fill="1" visible="yes" active="yes"/>
+<layer number="16" name="Bottom" color="2" fill="1" visible="yes" active="yes"/>
 <layer number="17" name="Pads" color="23" fill="1" visible="yes" active="yes"/>
 <layer number="18" name="Vias" color="29" fill="1" visible="yes" active="yes"/>
@@
 <text x="30.4198" y="75.311" size="3.81" layer="22" font="vector" ratio="20" rot="MR180">I2C-7313-IOB</text>
 <text x="22.622" y="56.642" size="1.4224" layer="22" font="vector" ratio="15" rot="MR344">Go Bears!</text>
-<text x="75.99675" y="60.80243125" size="1.27" layer="21" rot="SR0">16 bit I2C
+<text x="75.99675" y="64.61243125" size="1.27" layer="21" rot="SR0">16 bit I2C
 Digital I/O
 Active Low</text>
-<text x="76.34399375" y="83.389009375" size="1.016" layer="21">John Plocher</text>
+<text x="55.38899375" y="85.294009375" size="1.016" layer="21">John Plocher</text>
 <text x="81.8802" y="14.5034" size="1.016" layer="22" rot="SMR0">A "1" bit in the I/O register is associated with a LOW voltage on a pin,
 and a LIT feedback LED.</text>
@@
 <text x="8.41375" y="32.4485" size="1.016" layer="21" ratio="10" rot="R180">9 vDC</text>
 <text x="13.589" y="70.231" size="1.27" layer="21" rot="SR0">7805</text>
-<text x="77.35999375" y="68.339509375" size="1.016" layer="21">Hardware</text>
-<text x="76.34399375" y="77.610509375" size="1.016" layer="21">Open Source</text>
+<text x="78.62999375" y="78.499509375" size="1.016" layer="21">Hardware</text>
+<text x="77.61399375" y="86.500509375" size="1.016" layer="21">Open Source</text>
 <text x="1.27" y="103.505" size="1.016" layer="48">3.0A - Fixed C-POL, LED and VREG library component orientations to match default reel orientation, no PCB changes</text>
 <text x="0.889" y="17.399" size="1.27" layer="21">5v</text>
@@
 <text x="86.01339375" y="97.380534375" size="1.27" layer="21" rot="SR0">v3.1</text>
 <text x="85.48799375" y="95.645009375" size="1.016" layer="21">2020.08</text>
-<text x="53.73799375" y="80.405009375" size="1.016" layer="21">2018.01 1.0
+<text x="55.00799375" y="79.135009375" size="1.016" layer="21">2018.01 1.0
 2018.08 2.0
 2020.02 3.0
@@
 <attribute name="VALUE" x="50.38735" y="64.3254" size="0.8128" layer="27"/>
 </element>
-<element name="U$1" library="SparkFun" package="OSHW-LOGO-L" value="OSHW-LOGOL" x="80.645" y="72.517" smashed="yes"/>
+<element name="U$1" library="SparkFun" package="OSHW-LOGO-L" value="OSHW-LOGOL" x="81.915" y="82.677" smashed="yes"/>
 <element name="VR1" library="SPCoast" package="TO-252" value="CJ7805" x="13.335" y="78.74" smashed="yes">
 <attribute name="NAME" x="12.7" y="70.485" size="0.8128" layer="25" ratio="11" rot="R90"/>
@@
 </element>
 <element name="BOARD1" library="SPCoast" package="BOARD-DINRAIL-3.17IN-IOB" value="BOARD80X100-IOB" x="0" y="0"/>
-<element name="IOB1" library="SPCoast" package="IOB-IO4-CLEAN" value="CONNECTOR-IO4-IOBCLEAN" x="73.66" y="90.17" rot="R270"/>
-<element name="IOB2" library="SPCoast" package="IOB-IO4-CLEAN" value="CONNECTOR-IO4-IOBCLEAN" x="52.07" y="90.17" rot="R270"/>
-<element name="IOB3" library="SPCoast" package="IOB-IO4-CLEAN" value="CONNECTOR-IO4-IOBCLEAN" x="30.48" y="90.17" rot="R270"/>
-<element name="IOB4" library="SPCoast" package="IO4-IOB" value="CONNECTOR-IO4-IOBBARE" x="8.89" y="90.17" rot="R270"/>
-<element name="FID1" library="SPCoast" package="FIDUCIAL_1MM" value="FIDUCIAL" x="8.763" y="92.456"/>
-<element name="FID2" library="SPCoast" package="FIDUCIAL_1MM" value="FIDUCIAL" x="97.79" y="5.461"/>
+<element name="IOB1" library="SPCoast" package="IOB-IO4-NOBOTSILK" value="CONNECTOR-IO4-IOBNOBSILK" x="73.66" y="90.17" rot="R270"/>
+<element name="IOB2" library="SPCoast" package="IOB-IO4-NOBOTSILK" value="CONNECTOR-IO4-IOBNOBSILK" x="52.07" y="90.17" rot="R270"/>
+<element name="IOB3" library="SPCoast" package="IOB-IO4-NOBOTSILK" value="CONNECTOR-IO4-IOBNOBSILK" x="30.48" y="90.17" rot="R270"/>
+<element name="IOB4" library="SPCoast" package="IO4-IOB" value="CONNECTOR-IO4-IOBFULL" x="8.89" y="90.17" rot="R270"/>
+<element name="FID-UL" library="SPCoast" package="FIDUCIAL_1MM" value="FIDUCIAL" x="8.763" y="92.456" smashed="yes">
+<attribute name="NAME" x="10.668" y="92.456" size="1.016" layer="25"/>
+</element>
+<element name="FID-LR" library="SPCoast" package="FIDUCIAL_1MM" value="FIDUCIAL" x="97.79" y="5.461" smashed="yes">
+<attribute name="NAME" x="94.615" y="0.381" size="1.016" layer="25"/>
+</element>
 <element name="IC1" library="SPCoast" package="TSSOP24" value="MAX7311" x="51.435" y="57.15" smashed="yes" rot="R90">
 <attribute name="NAME" x="53.0225" y="59.3725" size="1.27" layer="25" rot="R180"/>
